Commit message: moved files around

File: rlbotics/envs/models/grippers/robotiq_2f_140/robotiq_2f_140.urdf (robot description, URDF)
Before this commit: robot robotiq_arg2f_140_model, 11 links, 10 joints
Links:
- link left_inner_finger: geometry collision mesh filename=meshes/collision/robotiq_arg2f_140_inner_finger.stl; visual mesh filename=meshes/visual/robotiq_arg2f_140_inner_finger.stl
- link left_inner_knuckle: geometry collision mesh filename=meshes/collision/robotiq_arg2f_140_inner_knuckle.stl; visual mesh filename=meshes/visual/robotiq_arg2f_140_inner_knuckle.stl
- link left_outer_finger: geometry collision mesh filename=meshes/collision/robotiq_arg2f_140_outer_finger.stl; visual mesh filename=meshes/visual/robotiq_arg2f_140_outer_finger.stl
- link left_outer_knuckle: geometry collision mesh filename=meshes/collision/robotiq_arg2f_140_outer_knuckle.stl; visual mesh filename=meshes/visual/robotiq_arg2f_140_outer_knuckle.stl
- link right_inner_finger: geometry collision mesh filename=meshes/collision/robotiq_arg2f_140_inner_finger.stl; visual mesh filename=meshes/visual/robotiq_arg2f_140_inner_finger.stl
- link right_inner_knuckle: geometry collision mesh filename=meshes/collision/robotiq_arg2f_140_inner_knuckle.stl; visual mesh filename=meshes/visual/robotiq_arg2f_140_inner_knuckle.stl
- link right_outer_finger: geometry collision mesh filename=meshes/collision/robotiq_arg2f_140_outer_finger.stl; visual mesh filename=meshes/visual/robotiq_arg2f_140_outer_finger.stl
- link right_outer_knuckle: geometry collision mesh filename=meshes/collision/robotiq_arg2f_140_outer_knuckle.stl; visual mesh filename=meshes/visual/robotiq_arg2f_140_outer_knuckle.stl
- link robotiq_arg2f_base_link: geometry collision mesh filename=meshes/collision/robotiq_arg2f_base_link.stl; visual mesh filename=meshes/visual/robotiq_arg2f_base_link.stl

File: rlbotics/envs/models/grippers/robotiq_2f_85/robotiq_2f_85.urdf (robot description, URDF)
Before this commit: robot robotiq_arg2f_85_model, 11 links, 10 joints
Links:
- link left_inner_finger: geometry collision mesh filename=meshes/collision/robotiq_arg2f_85_inner_finger.dae scale=0.001 0.001 0.001; visual mesh filename=meshes/visual/robotiq_arg2f_85_inner_finger.dae scale=0.001 0.001 0.001
- link left_inner_knuckle: geometry collision mesh filename=meshes/collision/robotiq_arg2f_85_inner_knuckle.dae scale=0.001 0.001 0.001; visual mesh filename=meshes/visual/robotiq_arg2f_85_inner_knuckle.dae scale=0.001 0.001 0.001
- link left_outer_finger: geometry collision mesh filename=meshes/collision/robotiq_arg2f_85_outer_finger.dae scale=0.001 0.001 0.001; visual mesh filename=meshes/visual/robotiq_arg2f_85_outer_finger.dae scale=0.001 0.001 0.001
- link left_outer_knuckle: geometry collision mesh filename=meshes/collision/robotiq_arg2f_85_outer_knuckle.dae scale=0.001 0.001 0.001; visual mesh filename=meshes/visual/robotiq_arg2f_85_outer_knuckle.dae scale=0.001 0.001 0.001
- link right_inner_finger: geometry collision mesh filename=meshes/collision/robotiq_arg2f_85_inner_finger.dae scale=0.001 0.001 0.001; visual mesh filename=meshes/visual/robotiq_arg2f_85_inner_finger.dae scale=0.001 0.001 0.001
- link right_inner_knuckle: geometry collision mesh filename=meshes/collision/robotiq_arg2f_85_inner_knuckle.dae scale=0.001 0.001 0.001; visual mesh filename=meshes/visual/robotiq_arg2f_85_inner_knuckle.dae scale=0.001 0.001 0.001
- link right_outer_finger: geometry collision mesh filename=meshes/collision/robotiq_arg2f_85_outer_finger.dae scale=0.001 0.001 0.001; visual mesh filename=meshes/visual/robotiq_arg2f_85_outer_finger.dae scale=0.001 0.001 0.001
- link right_outer_knuckle: geometry collision mesh filename=meshes/collision/robotiq_arg2f_85_outer_knuckle.dae scale=0.001 0.001 0.001; visual mesh filename=meshes/visual/robotiq_arg2f_85_outer_knuckle.dae scale=0.001 0.001 0.001
- link robotiq_arg2f_base_link: geometry collision mesh filename=meshes/collision/robotiq_arg2f_base_link.stl; visual mesh filename=meshes/visual/robotiq_arg2f_85_base_link.dae scale=0.001 0.001 0.001

File: rlbotics/envs/models/grippers/robotiq_3f/robotiq_3f.urdf (robot description, URDF)
Before this commit: robot robotiq-3f-gripper_articulated, 13 links, 12 joints
Links:
- link finger_1_link_0: geometry collision mesh filename=meshes/collision/link_0.STL; visual mesh filename=meshes/visual/link_0.dae
- link finger_1_link_1: geometry collision mesh filename=meshes/collision/link_1.STL; visual mesh filename=meshes/visual/link_1.dae
- link finger_1_link_2: geometry collision mesh filename=meshes/collision/link_2.STL; visual mesh filename=meshes/visual/link_2.dae
- link finger_1_link_3: geometry collision mesh filename=meshes/collision/link_3.STL; visual mesh filename=meshes/visual/link_3.dae
- link finger_2_link_0: geometry collision mesh filename=meshes/collision/link_0.STL; visual mesh filename=meshes/visual/link_0.dae
- link finger_2_link_1: geometry collision mesh filename=meshes/collision/link_1.STL; visual mesh filename=meshes/visual/link_1.dae
- link finger_2_link_2: geometry collision mesh filename=meshes/collision/link_2.STL; visual mesh filename=meshes/visual/link_2.dae
- link finger_2_link_3: geometry collision mesh filename=meshes/collision/link_3.STL; visual mesh filename=meshes/visual/link_3.dae
- link finger_middle_link_0: geometry collision mesh filename=meshes/collision/link_0.STL; visual mesh filename=meshes/visual/link_0.dae
- link finger_middle_link_1: geometry collision mesh filename=meshes/collision/link_1.STL; visual mesh filename=meshes/visual/link_1.dae
- link finger_middle_link_2: geometry collision mesh filename=meshes/collision/link_2.STL; visual mesh filename=meshes/visual/link_2.dae
- link finger_middle_link_3: geometry collision mesh filename=meshes/collision/link_3.STL; visual mesh filename=meshes/visual/link_3.dae
- link palm: geometry collision mesh filename=meshes/collision/palm.STL; visual mesh filename=meshes/visual/palm.dae

File: rlbotics/envs/models/robots/ur10/ur10.urdf (robot description, URDF)
Before this commit: robot ur10, 11 links, 10 joints
Links:
- link base_link: geometry collision mesh filename=meshes/collision/base.stl; visual mesh filename=meshes/visual/base.dae
- link forearm_link: geometry collision mesh filename=meshes/collision/forearm.stl; visual mesh filename=meshes/visual/forearm.dae
- link shoulder_link: geometry collision mesh filename=meshes/collision/shoulder.stl; visual mesh filename=meshes/visual/shoulder.dae
- link upper_arm_link: geometry collision mesh filename=meshes/collision/upperarm.stl; visual mesh filename=meshes/visual/upperarm.dae
- link wrist_1_link: geometry collision mesh filename=meshes/collision/wrist1.stl; visual mesh filename=meshes/visual/wrist1.dae
- link wrist_2_link: geometry collision mesh filename=meshes/collision/wrist2.stl; visual mesh filename=meshes/visual/wrist2.dae
- link wrist_3_link: geometry collision mesh filename=meshes/collision/wrist3.stl; visual mesh filename=meshes/visual/wrist3.dae
