Commit message: changed panda init pose

File: rlbotics/envs/models/misc/drill/drill.urdf (robot description, URDF)
Before this commit: robot drill, 1 links, 0 joints
Links:
- removed link root_link
- added link drillbit_bone, mass 0.001; collision box size=0.00279 0.00279 0.05353; visual mesh filename=meshes/dae/g_Drillbit_01.dae scale=0.07123 0.07123 0.07123
- added link grip_bone, mass 1.5; collision mesh filename=meshes/dae/g_g_carcaza_carcaza001.001.dae scale=0.07123 0.07123 0.07123; visual mesh filename=meshes/dae/g_g_carcaza_carcaza001.dae scale=0.07123 0.07123 0.07123
- added link root, mass 0.001; collision mesh filename=meshes/dae/g_g_taladro_taladro001.001.dae scale=0.24711 0.24711 0.24711; collision mesh filename=meshes/dae/meshId5_name.001.dae scale=0.24711 0.24711 0.24711
Joints:
- added joint drillbit_bone: type fixed, parent root, child drillbit_bone, origin xyz=0.00052 0.00107 -0.18095 rpy=3.14159 0 0
- added joint grip_bone: type fixed, parent root, child grip_bone, origin xyz=0.00063 0.03195 -0.02401 rpy=1.5708 0 0

Commit message: edited drill model

File: rlbotics/envs/models/misc/drill/drill.urdf (robot description, URDF)
Before this commit: robot drill, 3 links, 2 joints
Links:
- link drillbit_bone: geometry collision box size=0.00279 0.00279 0.05353; visual mesh filename=meshes/g_Drillbit_01.dae scale=0.07123 0.07123 0.07123
- link grip_bone: geometry collision mesh filename=meshes/g_g_carcaza_carcaza001.001.dae scale=0.07123 0.07123 0.07123; visual mesh filename=meshes/g_g_carcaza_carcaza001.dae scale=0.07123 0.07123 0.07123
- link root: geometry collision mesh filename=meshes/g_g_taladro_taladro001.001.dae scale=0.24711 0.24711 0.24711; collision mesh filename=meshes/meshId5_name.001.dae scale=0.24711 0.24711 0.24711
Joints:
- joint grip_bone: origin xyz=0.00063 0.03195 -0.02401 rpy=1.5708 0 0 -> xyz=0.00063 0.03473 -0.02401 rpy=1.5708 0 0

Commit message: made new file structure for robots and grippers

File: rlbotics/envs/models/misc/drill/drill.urdf (robot description, URDF)
Before this commit: robot drill, 3 links, 2 joints
Links:
- link drillbit_bone: geometry collision box size=0.00279 0.00279 0.05353; visual mesh filename=meshes/dae/g_Drillbit_01.dae scale=0.07123 0.07123 0.07123
- link grip_bone: geometry collision mesh filename=meshes/dae/g_g_carcaza_carcaza001.001.dae scale=0.07123 0.07123 0.07123; visual mesh filename=meshes/dae/g_g_carcaza_carcaza001.dae scale=0.07123 0.07123 0.07123
- link root: geometry collision mesh filename=meshes/dae/g_g_taladro_taladro001.001.dae scale=0.24711 0.24711 0.24711; collision mesh filename=meshes/dae/meshId5_name.001.dae scale=0.24711 0.24711 0.24711

File: rlbotics/envs/models/misc/drill/drill_old.urdf (robot description, URDF)
Before this commit: robot drill, 3 links, 2 joints
Joints:
- joint grip_bone: origin xyz=0.00063 0.03195 -0.02401 rpy=1.5708 0 0 -> xyz=0.00063 0.03473 -0.02401 rpy=1.5708 0 0
