Commit message: trial

File: rlbotics/envs/models/combined/ur10_robotiq_2f_85.urdf (robot description, URDF)
Before this commit: robot , 22 links, 21 joints
Links:
- link base_link: geometry collision mesh filename=rlbotics/envs/models/robots/universal_robots/ur10/meshes/co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 scale=1.00000 1.00000 1.00000; visual mesh filename=rlbotics/envs/models/robots/universal_robots/ur10/meshes/vi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 scale=1.00000 1.00000 1.00000
- link forearm_link: geometry collision mesh filename=rlbotics/envs/models/robots/universal_robots/ur10/meshes/co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 scale=1.00000 1.00000 1.00000; visual mesh filename=rlbotics/envs/models/robots/universal_robots/ur10/meshes/vi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 scale=1.00000 1.00000 1.00000
- link left_inner_finger: geometry collision mesh filename=rlbotics/envs/models/grippers/robotiq/robotiq_2f_85/meshes/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 scale=0.00100 0.00100 0.00100; visual mesh filename=rlbotics/envs/models/grippers/robotiq/robotiq_2f_85/meshes/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 scale=0.00100 0.00100 0.00100
- link left_inner_knuckle: geometry collision mesh filename=rlbotics/envs/models/grippers/robotiq/robotiq_2f_85/meshes/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 scale=0.00100 0.00100 0.00100; visual mesh filename=rlbotics/envs/models/grippers/robotiq/robotiq_2f_85/meshes/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 scale=0.00100 0.00100 0.00100
- link left_outer_finger: geometry collision mesh filename=rlbotics/envs/models/grippers/robotiq/robotiq_2f_85/meshes/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 scale=0.00100 0.00100 0.00100; visual mesh filename=rlbotics/envs/models/grippers/robotiq/robotiq_2f_85/meshes/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 scale=0.00100 0.00100 0.00100
- link left_outer_knuckle: geometry collision mesh filename=rlbotics/envs/models/grippers/robotiq/robotiq_2f_85/meshes/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 scale=0.00100 0.00100 0.00100; visual mesh filename=rlbotics/envs/models/grippers/robotiq/robotiq_2f_85/meshes/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 scale=0.00100 0.00100 0.00100
- link right_inner_finger: geometry collision mesh filename=rlbotics/envs/models/grippers/robotiq/robotiq_2f_85/meshes/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 scale=0.00100 0.00100 0.00100; visual mesh filename=rlbotics/envs/models/grippers/robotiq/robotiq_2f_85/meshes/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 scale=0.00100 0.00100 0.00100
- link right_inner_knuckle: geometry collision mesh filename=rlbotics/envs/models/grippers/robotiq/robotiq_2f_85/meshes/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 scale=0.00100 0.00100 0.00100; visual mesh filename=rlbotics/envs/models/grippers/robotiq/robotiq_2f_85/meshes/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 scale=0.00100 0.00100 0.00100
- link right_outer_finger: geometry collision mesh filename=rlbotics/envs/models/grippers/robotiq/robotiq_2f_85/meshes/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 scale=0.00100 0.00100 0.00100; visual mesh filename=rlbotics/envs/models/grippers/robotiq/robotiq_2f_85/meshes/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 scale=0.00100 0.00100 0.00100
- link right_outer_knuckle: geometry collision mesh filename=rlbotics/envs/models/grippers/robotiq/robotiq_2f_85/meshes/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 scale=0.00100 0.00100 0.00100; visual mesh filename=rlbotics/envs/models/grippers/robotiq/robotiq_2f_85/meshes/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 scale=0.00100 0.00100 0.00100
- link robotiq_arg2f_base_link: geometry collision mesh filename=rlbotics/envs/models/grippers/robotiq/robotiq_2f_85/meshes/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 scale=1.00000 1.00000 1.00000; visual mesh filename=rlbotics/envs/models/grippers/robotiq/robotiq_2f_85/meshes/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 scale=0.00100 0.00100 0.00100
- link shoulder_link: geometry collision mesh filename=rlbotics/envs/models/robots/universal_robots/ur10/meshes/co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 scale=1.00000 1.00000 1.00000; visual mesh filename=rlbotics/envs/models/robots/universal_robots/ur10/meshes/vi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 scale=1.00000 1.00000 1.00000
- link upper_arm_link: geometry collision mesh filename=rlbotics/envs/models/robots/universal_robots/ur10/meshes/co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 scale=1.00000 1.00000 1.00000; visual mesh filename=rlbotics/envs/models/robots/universal_robots/ur10/meshes/vi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 scale=1.00000 1.00000 1.00000
- link wrist_1_link: geometry collision mesh filename=rlbotics/envs/models/robots/universal_robots/ur10/meshes/co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 scale=1.00000 1.00000 1.00000; visual mesh filename=rlbotics/envs/models/robots/universal_robots/ur10/meshes/vi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 scale=1.00000 1.00000 1.00000
- link wrist_2_link: geometry collision mesh filename=rlbotics/envs/models/robots/universal_robots/ur10/meshes/co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 scale=1.00000 1.00000 1.00000; visual mesh filename=rlbotics/envs/models/robots/universal_robots/ur10/meshes/vi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 scale=1.00000 1.00000 1.00000
- link wrist_3_link: geometry collision mesh filename=rlbotics/envs/models/robots/universal_robots/ur10/meshes/co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 scale=1.00000 1.00000 1.00000; visual mesh filename=rlbotics/envs/models/robots/universal_robots/ur10/meshes/vi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 scale=1.00000 1.00000 1.00000

Commit message: combining urdf fix.

File: rlbotics/envs/models/combined/ur10_robotiq_2f_85.urdf (robot description, URDF)
Before this commit: robot , 22 links, 21 joints
Joints:
- joint elbow_joint: limit (none) -> lower=-3.141592653589793 upper=3.141592653589793 effort=150.0 velocity=3.15; type continuous -> revolute
- joint finger_joint: limit (none) -> lower=0.0 upper=0.8 effort=1000.0 velocity=2.0; type continuous -> revolute
- joint left_inner_finger_joint: limit (none) -> lower=0.0 upper=0.8757 effort=1000.0 velocity=2.0; type continuous -> revolute
- joint left_inner_knuckle_joint: limit (none) -> lower=0.0 upper=0.8757 effort=1000.0 velocity=2.0; type continuous -> revolute
- joint right_inner_finger_joint: limit (none) -> lower=0.0 upper=0.8757 effort=1000.0 velocity=2.0; type continuous -> revolute
- joint right_inner_knuckle_joint: limit (none) -> lower=0.0 upper=0.8757 effort=1000.0 velocity=2.0; type continuous -> revolute
- joint right_outer_knuckle_joint: limit (none) -> lower=0.0 upper=0.81 effort=1000.0 velocity=2.0; type continuous -> revolute
- joint shoulder_lift_joint: limit (none) -> lower=-6.283185307179586 upper=6.283185307179586 effort=330.0 velocity=2.16; type continuous -> revolute
- joint shoulder_pan_joint: limit (none) -> lower=-6.283185307179586 upper=6.283185307179586 effort=330.0 velocity=2.16; type continuous -> revolute
- joint wrist_1_joint: limit (none) -> lower=-6.283185307179586 upper=6.283185307179586 effort=54.0 velocity=3.2; type continuous -> revolute
- joint wrist_2_joint: limit (none) -> lower=-6.283185307179586 upper=6.283185307179586 effort=54.0 velocity=3.2; type continuous -> revolute
- joint wrist_3_joint: limit (none) -> lower=-6.283185307179586 upper=6.283185307179586 effort=54.0 velocity=3.2; type continuous -> revolute
