Commit message: scaled up welding torch

File: rlbotics/envs/models/combined/ur10_welding_torch.urdf (robot description, URDF)
Before this commit: robot , 14 links, 13 joints
Links:
- link ee_joint_arm: geometry collision mesh filename=rlbotics/envs/models/end_effectors/welding_torches/welding_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 scale=1.91308 1.91308 1.91308; visual mesh filename=rlbotics/envs/models/end_effectors/welding_torches/welding_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 scale=0.01913 0.01913 0.01913
- link nozzle_tip: geometry collision mesh filename=rlbotics/envs/models/end_effectors/welding_torches/welding_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 scale=1.91308 1.91308 1.91308; visual mesh filename=rlbotics/envs/models/end_effectors/welding_torches/welding_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 scale=0.01913 0.01913 0.01913
- link root: geometry collision mesh filename=rlbotics/envs/models/end_effectors/welding_torches/welding_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 scale=1.91308 1.91308 1.91308; collision mesh filename=rlbotics/envs/models/end_effectors/welding_torches/welding_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 scale=1.91308 1.91308 1.91308
Joints:
- joint ee_joint_arm: origin xyz=0.00003 0.00159 -0.02985 rpy=0.00000 -0.00000 0.00000 -> xyz=0.00005 0.00304 -0.05711 rpy=0.00000 -0.00000 0.00000
- joint joint_dummy1: origin xyz=0.00000 0.00000 0.00000 rpy=3.14159 1.57080 0.00000 -> xyz=0.00000 0.00000 0.00000 rpy=0.00000 1.57080 0.00000
- joint nozzle_tip: origin xyz=0.00101 0.00731 0.39981 rpy=0.92502 -0.00000 0.00000 -> xyz=0.00193 0.01399 0.76487 rpy=0.92502 -0.00000 0.00000

File: rlbotics/envs/models/end_effectors/welding_torches/welding_torch/welding_torch.urdf (robot description, URDF)
Before this commit: robot welding_torch, 3 links, 2 joints
Links:
- link ee_joint_arm: geometry collision mesh filename=meshes/stl/Body22.001.stl scale=1.91308 1.91308 1.91308; visual mesh filename=meshes/stl/Body22.stl scale=0.01913 0.01913 0.01913
- link nozzle_tip: geometry collision mesh filename=meshes/stl/Body28.001.stl scale=1.91308 1.91308 1.91308; visual mesh filename=meshes/stl/Body28.stl scale=0.01913 0.01913 0.01913
- link root: geometry collision mesh filename=meshes/stl/Body1.001.stl scale=1.91308 1.91308 1.91308; collision mesh filename=meshes/stl/Body23.001.stl scale=1.91308 1.91308 1.91308
Joints:
- joint ee_joint_arm: origin xyz=3e-05 0.00159 -0.02985 rpy=0 0 0 -> xyz=5e-05 0.00304 -0.05711 rpy=0 0 0
- joint nozzle_tip: origin xyz=0.00101 0.00731 0.39981 rpy=0.92502 0 0 -> xyz=0.00193 0.01399 0.76487 rpy=0.92502 0 0
