Commit message: IK testing script in load_manipulator.py

File: rlbotics/envs/models/combined/abb_irb6640_welding_torch.urdf (robot description, URDF)
Before this commit: robot , 14 links, 13 joints
Links:
- link ee_joint_arm: geometry collision mesh filename=rlbotics/envs/models/end_effectors/welding/welding_torch/me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 scale=1.91308 1.91308 1.91308; visual mesh filename=rlbotics/envs/models/end_effectors/welding/welding_torch/me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 scale=0.01913 0.01913 0.01913
- link nozzle_tip: geometry collision mesh filename=rlbotics/envs/models/end_effectors/welding/welding_torch/me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 scale=1.91308 1.91308 1.91308; visual mesh filename=rlbotics/envs/models/end_effectors/welding/welding_torch/me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 scale=0.01913 0.01913 0.01913
- link root: geometry collision mesh filename=rlbotics/envs/models/end_effectors/welding/welding_torch/me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 scale=1.91308 1.91308 1.91308; collision mesh filename=rlbotics/envs/models/end_effectors/welding/welding_torch/me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 scale=1.91308 1.91308 1.91308
Joints:
- joint ee_joint_arm: origin xyz=0.00004 0.00232 -0.04351 rpy=0.00000 -0.00000 0.00000 -> xyz=0.00005 0.00304 -0.05711 rpy=0.00000 -0.00000 0.00000
- joint nozzle_tip: origin xyz=0.00147 0.01066 0.58278 rpy=0.92502 -0.00000 0.00000 -> xyz=0.00193 0.01399 0.76487 rpy=0.92502 -0.00000 0.00000

File: rlbotics/envs/models/combined/kuka_kr210l150_welding_torch.urdf (robot description, URDF)
Before this commit: robot , 12 links, 11 joints
Links:
- link ee_joint_arm: geometry collision mesh filename=rlbotics/envs/models/end_effectors/welding/welding_torch/me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 scale=1.91308 1.91308 1.91308; visual mesh filename=rlbotics/envs/models/end_effectors/welding/welding_torch/me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 scale=0.01913 0.01913 0.01913
- link nozzle_tip: geometry collision mesh filename=rlbotics/envs/models/end_effectors/welding/welding_torch/me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 scale=1.91308 1.91308 1.91308; visual mesh filename=rlbotics/envs/models/end_effectors/welding/welding_torch/me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 scale=0.01913 0.01913 0.01913
- link root: geometry collision mesh filename=rlbotics/envs/models/end_effectors/welding/welding_torch/me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 scale=1.91308 1.91308 1.91308; collision mesh filename=rlbotics/envs/models/end_effectors/welding/welding_torch/me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 scale=1.91308 1.91308 1.91308

File: rlbotics/envs/models/combined/ur10_robotiq_2f_85.urdf (robot description, URDF)
Before this commit: robot , 22 links, 21 joints
Links:
- link base_link: geometry collision mesh filename=rlbotics/envs/models/robots/universal_robots/ur10/meshes/ur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 scale=1.00000 1.00000 1.00000; visual mesh filename=rlbotics/envs/models/robots/universal_robots/ur10/meshes/ur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 scale=1.00000 1.00000 1.00000
- link forearm_link: geometry collision mesh filename=rlbotics/envs/models/robots/universal_robots/ur10/meshes/ur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 scale=1.00000 1.00000 1.00000; visual mesh filename=rlbotics/envs/models/robots/universal_robots/ur10/meshes/ur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 scale=1.00000 1.00000 1.00000
- link left_inner_finger: geometry collision mesh filename=rlbotics/envs/models/end_effectors/robotiq/robotiq_2f_85/me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 scale=0.00100 0.00100 0.00100; visual mesh filename=rlbotics/envs/models/end_effectors/robotiq/robotiq_2f_85/me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 scale=0.00100 0.00100 0.00100
- link left_inner_knuckle: geometry collision mesh filename=rlbotics/envs/models/end_effectors/robotiq/robotiq_2f_85/me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 scale=0.00100 0.00100 0.00100; visual mesh filename=rlbotics/envs/models/end_effectors/robotiq/robotiq_2f_85/me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 scale=0.00100 0.00100 0.00100
- link left_outer_finger: geometry collision mesh filename=rlbotics/envs/models/end_effectors/robotiq/robotiq_2f_85/me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 scale=0.00100 0.00100 0.00100; visual mesh filename=rlbotics/envs/models/end_effectors/robotiq/robotiq_2f_85/me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 scale=0.00100 0.00100 0.00100
- link left_outer_knuckle: geometry collision mesh filename=rlbotics/envs/models/end_effectors/robotiq/robotiq_2f_85/me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 scale=0.00100 0.00100 0.00100; visual mesh filename=rlbotics/envs/models/end_effectors/robotiq/robotiq_2f_85/me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 scale=0.00100 0.00100 0.00100
- link right_inner_finger: geometry collision mesh filename=rlbotics/envs/models/end_effectors/robotiq/robotiq_2f_85/me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 scale=0.00100 0.00100 0.00100; visual mesh filename=rlbotics/envs/models/end_effectors/robotiq/robotiq_2f_85/me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 scale=0.00100 0.00100 0.00100
- link right_inner_knuckle: geometry collision mesh filename=rlbotics/envs/models/end_effectors/robotiq/robotiq_2f_85/me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 scale=0.00100 0.00100 0.00100; visual mesh filename=rlbotics/envs/models/end_effectors/robotiq/robotiq_2f_85/me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 scale=0.00100 0.00100 0.00100
- link right_outer_finger: geometry collision mesh filename=rlbotics/envs/models/end_effectors/robotiq/robotiq_2f_85/me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 scale=0.00100 0.00100 0.00100; visual mesh filename=rlbotics/envs/models/end_effectors/robotiq/robotiq_2f_85/me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 scale=0.00100 0.00100 0.00100
- link right_outer_knuckle: geometry collision mesh filename=rlbotics/envs/models/end_effectors/robotiq/robotiq_2f_85/me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 scale=0.00100 0.00100 0.00100; visual mesh filename=rlbotics/envs/models/end_effectors/robotiq/robotiq_2f_85/me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 scale=0.00100 0.00100 0.00100
- link robotiq_arg2f_base_link: geometry collision mesh filename=rlbotics/envs/models/end_effectors/robotiq/robotiq_2f_85/me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 scale=1.00000 1.00000 1.00000; visual mesh filename=rlbotics/envs/models/end_effectors/robotiq/robotiq_2f_85/me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 scale=0.00100 0.00100 0.00100
- link shoulder_link: geometry collision mesh filename=rlbotics/envs/models/robots/universal_robots/ur10/meshes/ur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 scale=1.00000 1.00000 1.00000; visual mesh filename=rlbotics/envs/models/robots/universal_robots/ur10/meshes/ur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 scale=1.00000 1.00000 1.00000
- link upper_arm_link: geometry collision mesh filename=rlbotics/envs/models/robots/universal_robots/ur10/meshes/ur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 scale=1.00000 1.00000 1.00000; visual mesh filename=rlbotics/envs/models/robots/universal_robots/ur10/meshes/ur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 scale=1.00000 1.00000 1.00000
- link wrist_1_link: geometry collision mesh filename=rlbotics/envs/models/robots/universal_robots/ur10/meshes/ur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 scale=1.00000 1.00000 1.00000; visual mesh filename=rlbotics/envs/models/robots/universal_robots/ur10/meshes/ur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 scale=1.00000 1.00000 1.00000
- link wrist_2_link: geometry collision mesh filename=rlbotics/envs/models/robots/universal_robots/ur10/meshes/ur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 scale=1.00000 1.00000 1.00000; visual mesh filename=rlbotics/envs/models/robots/universal_robots/ur10/meshes/ur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 scale=1.00000 1.00000 1.00000
- link wrist_3_link: geometry collision mesh filename=rlbotics/envs/models/robots/universal_robots/ur10/meshes/ur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 scale=1.00000 1.00000 1.00000; visual mesh filename=rlbotics/envs/models/robots/universal_robots/ur10/meshes/ur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 scale=1.00000 1.00000 1.00000

File: rlbotics/envs/models/combined/ur10_welding_torch.urdf (robot description, URDF)
Before this commit: robot , 14 links, 13 joints
Links:
- link ee_joint_arm: geometry collision mesh filename=rlbotics/envs/models/end_effectors/welding/welding_torch/me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 scale=1.91308 1.91308 1.91308; visual mesh filename=rlbotics/envs/models/end_effectors/welding/welding_torch/me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 scale=0.01913 0.01913 0.01913
- link nozzle_tip: geometry collision mesh filename=rlbotics/envs/models/end_effectors/welding/welding_torch/me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 scale=1.91308 1.91308 1.91308; visual mesh filename=rlbotics/envs/models/end_effectors/welding/welding_torch/me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 scale=0.01913 0.01913 0.01913
- link root: geometry collision mesh filename=rlbotics/envs/models/end_effectors/welding/welding_torch/me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 scale=1.91308 1.91308 1.91308; collision mesh filename=rlbotics/envs/models/end_effectors/welding/welding_torch/me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 scale=1.91308 1.91308 1.91308
