Commit message: spot welding gun in body in white world

File: rlbotics/envs/models/combined/abb_irb6640_spot_welding_gun.urdf (robot description, URDF)
Before this commit: robot , 14 links, 13 joints
Links:
- link base_link: geometry collision mesh filename=rlbotics\envs\models\robots/abb/irb6600/meshes/irb6640/coll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 scale=1.00000 1.00000 1.00000; visual mesh filename=rlbotics\envs\models\robots/abb/irb6600/meshes/irb6640/visu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 scale=1.00000 1.00000 1.00000
- link link_1: geometry collision mesh filename=rlbotics\envs\models\robots/abb/irb6600/meshes/irb6640/coll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 scale=1.00000 1.00000 1.00000; visual mesh filename=rlbotics\envs\models\robots/abb/irb6600/meshes/irb6640/visu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 scale=1.00000 1.00000 1.00000
- link link_2: geometry collision mesh filename=rlbotics\envs\models\robots/abb/irb6600/meshes/irb6640/coll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 scale=1.00000 1.00000 1.00000; visual mesh filename=rlbotics\envs\models\robots/abb/irb6600/meshes/irb6640/visu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 scale=1.00000 1.00000 1.00000
- link link_3: geometry collision mesh filename=rlbotics\envs\models\robots/abb/irb6600/meshes/irb6640/coll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 scale=1.00000 1.00000 1.00000; visual mesh filename=rlbotics\envs\models\robots/abb/irb6600/meshes/irb6640/visu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 scale=1.00000 1.00000 1.00000
- link link_4: geometry collision mesh filename=rlbotics\envs\models\robots/abb/irb6600/meshes/irb6640/coll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 scale=1.00000 1.00000 1.00000; visual mesh filename=rlbotics\envs\models\robots/abb/irb6600/meshes/irb6640/visu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 scale=1.00000 1.00000 1.00000
- link link_5: geometry collision mesh filename=rlbotics\envs\models\robots/abb/irb6600/meshes/irb6640/coll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 scale=1.00000 1.00000 1.00000; visual mesh filename=rlbotics\envs\models\robots/abb/irb6600/meshes/irb6640/visu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 scale=1.00000 1.00000 1.00000
- link link_6: geometry collision mesh filename=rlbotics\envs\models\robots/abb/irb6600/meshes/irb6640/coll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 scale=1.00000 1.00000 1.00000; visual mesh filename=rlbotics\envs\models\robots/abb/irb6600/meshes/irb6640/visu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 scale=1.00000 1.00000 1.00000
- link link_cylinder: geometry collision mesh filename=rlbotics\envs\models\robots/abb/irb6600/meshes/irb6640/coll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 scale=1.00000 1.00000 1.00000; visual mesh filename=rlbotics\envs\models\robots/abb/irb6600/meshes/irb6640/visu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 scale=1.00000 1.00000 1.00000
- link link_piston: geometry collision mesh filename=rlbotics\envs\models\robots/abb/irb6600/meshes/irb6640/coll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 scale=1.00000 1.00000 1.00000; visual mesh filename=rlbotics\envs\models\robots/abb/irb6600/meshes/irb6640/visu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 scale=1.00000 1.00000 1.00000
- link root: geometry collision mesh filename=rlbotics\envs\models\end_effectors/welding/spot_welding_gun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 scale=0.78991 0.78991 0.78991; visual mesh filename=rlbotics\envs\models\end_effectors/welding/spot_welding_gun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 scale=0.00116 0.00116 0.00116

File: rlbotics/envs/models/misc/world_plane/plane.urdf (robot description, URDF)
Before this commit: robot plane, 1 links, 0 joints
Links:
- removed link planeLink
- added link plane_link, mass .0; collision box size=20 20 0.1; visual box size=20 20 0.1
