Commit message: fixed robot urdf file structure to be consistent

File: rlbotics/envs/models/robots/fanuc/cr35ia/cr35ia.urdf (robot description, URDF)
Before this commit: robot fanuc_cr35ia, 10 links, 9 joints
Links:
- link base_link: geometry collision mesh filename=meshes/cr35ia/collision/base_link.stl; visual mesh filename=meshes/cr35ia/visual/base_link.stl
- link link_1: geometry collision mesh filename=meshes/cr35ia/collision/link_1.stl; visual mesh filename=meshes/cr35ia/visual/link_1.stl
- link link_2: geometry collision mesh filename=meshes/cr35ia/collision/link_2.stl; visual mesh filename=meshes/cr35ia/visual/link_2.stl
- link link_3: geometry collision mesh filename=meshes/cr35ia/collision/link_3.stl; visual mesh filename=meshes/cr35ia/visual/link_3.stl
- link link_4: geometry collision mesh filename=meshes/cr35ia/collision/link_4.stl; visual mesh filename=meshes/cr35ia/visual/link_4.stl
- link link_5: geometry collision mesh filename=meshes/cr35ia/collision/link_5.stl; visual mesh filename=meshes/cr35ia/visual/link_5.stl
- link link_6: geometry collision mesh filename=meshes/cr35ia/collision/link_6.stl; visual mesh filename=meshes/cr35ia/visual/link_6.stl

File: rlbotics/envs/models/robots/fanuc/lrmate200i/lrmate200i.urdf (robot description, URDF)
Before this commit: robot fanuc_lrmate200i, 10 links, 9 joints
Links:
- link base_link: geometry collision mesh filename=meshes/lrmate200i/collision/base_link.stl; visual mesh filename=meshes/lrmate200i/visual/base_link.stl
- link link_1: geometry collision mesh filename=meshes/lrmate200i/collision/link_1.stl; visual mesh filename=meshes/lrmate200i/visual/link_1.stl
- link link_2: geometry collision mesh filename=meshes/lrmate200i/collision/link_2.stl; visual mesh filename=meshes/lrmate200i/visual/link_2.stl
- link link_3: geometry collision mesh filename=meshes/lrmate200i/collision/link_3.stl; visual mesh filename=meshes/lrmate200i/visual/link_3.stl
- link link_4: geometry collision mesh filename=meshes/lrmate200i/collision/link_4.stl; visual mesh filename=meshes/lrmate200i/visual/link_4.stl
- link link_5: geometry collision mesh filename=meshes/lrmate200i/collision/link_5.stl; visual mesh filename=meshes/lrmate200i/visual/link_5.stl
- link link_6: geometry collision mesh filename=meshes/lrmate200i/collision/link_6.stl; visual mesh filename=meshes/lrmate200i/visual/link_6.stl

File: rlbotics/envs/models/robots/fanuc/m16ib/m16ib20.urdf (robot description, URDF)
Before this commit: robot fanuc_m16ib20, 10 links, 9 joints
Links:
- link base_link: geometry collision mesh filename=meshes/m16ib20/collision/base_link.stl; visual mesh filename=meshes/m16ib20/visual/base_link.stl
- link link_1: geometry collision mesh filename=meshes/m16ib20/collision/link_1.stl; visual mesh filename=meshes/m16ib20/visual/link_1.stl
- link link_2: geometry collision mesh filename=meshes/m16ib20/collision/link_2.stl; visual mesh filename=meshes/m16ib20/visual/link_2.stl
- link link_3: geometry collision mesh filename=meshes/m16ib20/collision/link_3.stl; visual mesh filename=meshes/m16ib20/visual/link_3.stl
- link link_4: geometry collision mesh filename=meshes/m16ib20/collision/link_4.stl; visual mesh filename=meshes/m16ib20/visual/link_4.stl
- link link_5: geometry collision mesh filename=meshes/m16ib20/collision/link_5.stl; visual mesh filename=meshes/m16ib20/visual/link_5.stl
- link link_6: geometry collision mesh filename=meshes/m16ib20/collision/link_6.stl; visual mesh filename=meshes/m16ib20/visual/link_6.stl

File: rlbotics/envs/models/robots/fanuc/m20ib/m20ib25.urdf (robot description, URDF)
Before this commit: robot fanuc_m20ib25, 10 links, 9 joints
Links:
- link base_link: geometry collision mesh filename=meshes/m20ib25/collision/base_link.stl; visual mesh filename=meshes/m20ib25/visual/base_link.stl
- link link_1: geometry collision mesh filename=meshes/m20ib25/collision/link_1.stl; visual mesh filename=meshes/m20ib25/visual/link_1.stl
- link link_2: geometry collision mesh filename=meshes/m20ib25/collision/link_2.stl; visual mesh filename=meshes/m20ib25/visual/link_2.stl
- link link_3: geometry collision mesh filename=meshes/m20ib25/collision/link_3.stl; visual mesh filename=meshes/m20ib25/visual/link_3.stl
- link link_4: geometry collision mesh filename=meshes/m20ib25/collision/link_4.stl; visual mesh filename=meshes/m20ib25/visual/link_4.stl
- link link_5: geometry collision mesh filename=meshes/m20ib25/collision/link_5.stl; visual mesh filename=meshes/m20ib25/visual/link_5.stl
- link link_6: geometry collision mesh filename=meshes/m20ib25/collision/link_6.stl; visual mesh filename=meshes/m20ib25/visual/link_6.stl

File: rlbotics/envs/models/robots/fanuc/m900ia/m900ia260l.urdf (robot description, URDF)
Before this commit: robot fanuc_m900ia260l, 12 links, 11 joints
Links:
- link base_link: geometry collision mesh filename=meshes/m900ia260l/collision/base_link.stl; visual mesh filename=meshes/m900ia260l/visual/base_link.stl
- link link_1: geometry collision mesh filename=meshes/m900ia260l/collision/link_1.stl; visual mesh filename=meshes/m900ia260l/visual/link_1.stl
- link link_2: geometry collision mesh filename=meshes/m900ia260l/collision/link_2.stl; visual mesh filename=meshes/m900ia260l/visual/link_2.stl
- link link_3: geometry collision mesh filename=meshes/m900ia260l/collision/link_3.stl; visual mesh filename=meshes/m900ia260l/visual/link_3.stl
- link link_4: geometry collision mesh filename=meshes/m900ia260l/collision/link_4.stl; visual mesh filename=meshes/m900ia260l/visual/link_4.stl
- link link_5: geometry collision mesh filename=meshes/m900ia260l/collision/link_5.stl; visual mesh filename=meshes/m900ia260l/visual/link_5.stl
- link link_6: geometry collision mesh filename=meshes/m900ia260l/collision/link_6.stl; visual mesh filename=meshes/m900ia260l/visual/link_6.stl
- link plink_1: geometry collision mesh filename=meshes/m900ia260l/collision/plink_1.stl; visual mesh filename=meshes/m900ia260l/visual/plink_1.stl
- link plink_2: geometry collision mesh filename=meshes/m900ia260l/collision/plink_2.stl; visual mesh filename=meshes/m900ia260l/visual/plink_2.stl

File: rlbotics/envs/models/robots/fanuc/m900ib/m900ib700.urdf (robot description, URDF)
Before this commit: robot fanuc_m900ib700, 16 links, 15 joints
Links:
- link balancer_left: geometry collision mesh filename=meshes/m900ib700/collision/balancer.stl; visual mesh filename=meshes/m900ib700/visual/balancer.stl
- link balancer_right: geometry collision mesh filename=meshes/m900ib700/collision/balancer.stl; visual mesh filename=meshes/m900ib700/visual/balancer.stl
- link base_link: geometry collision mesh filename=meshes/m900ib700/collision/base_link.stl; visual mesh filename=meshes/m900ib700/visual/base_link.stl
- link link_1: geometry collision mesh filename=meshes/m900ib700/collision/link_1.stl; visual mesh filename=meshes/m900ib700/visual/link_1.stl
- link link_2: geometry collision mesh filename=meshes/m900ib700/collision/link_2.stl; visual mesh filename=meshes/m900ib700/visual/link_2.stl
- link link_3: geometry collision mesh filename=meshes/m900ib700/collision/link_3.stl; visual mesh filename=meshes/m900ib700/visual/link_3.stl
- link link_4: geometry collision mesh filename=meshes/m900ib700/collision/link_4.stl; visual mesh filename=meshes/m900ib700/visual/link_4.stl
- link link_5: geometry collision mesh filename=meshes/m900ib700/collision/link_5.stl; visual mesh filename=meshes/m900ib700/visual/link_5.stl
- link link_6: geometry collision mesh filename=meshes/m900ib700/collision/link_6.stl; visual mesh filename=meshes/m900ib700/visual/link_6.stl
- link piston_left: geometry collision mesh filename=meshes/m900ib700/collision/piston.stl; visual mesh filename=meshes/m900ib700/visual/piston.stl
- link piston_right: geometry collision mesh filename=meshes/m900ib700/collision/piston.stl; visual mesh filename=meshes/m900ib700/visual/piston.stl
- link plink_1: geometry collision mesh filename=meshes/m900ib700/collision/counterweight.stl; visual mesh filename=meshes/m900ib700/visual/counterweight.stl
- link plink_2: geometry collision mesh filename=meshes/m900ib700/collision/bar.stl; visual mesh filename=meshes/m900ib700/visual/bar.stl

File: rlbotics/envs/models/robots/fanuc/r1000ia/r1000ia80f.urdf (robot description, URDF)
Before this commit: robot fanuc_r1000ia80f, 10 links, 9 joints
Links:
- link base_link: geometry collision mesh filename=meshes/r1000ia80f/collision/base_link.stl; visual mesh filename=meshes/r1000ia80f/visual/base_link.stl
- link link_1: geometry collision mesh filename=meshes/r1000ia80f/collision/link_1.stl; visual mesh filename=meshes/r1000ia80f/visual/link_1.stl
- link link_2: geometry collision mesh filename=meshes/r1000ia80f/collision/link_2.stl; visual mesh filename=meshes/r1000ia80f/visual/link_2.stl
- link link_3: geometry collision mesh filename=meshes/r1000ia80f/collision/link_3.stl; visual mesh filename=meshes/r1000ia80f/visual/link_3.stl
- link link_4: geometry collision mesh filename=meshes/r1000ia80f/collision/link_4.stl; visual mesh filename=meshes/r1000ia80f/visual/link_4.stl
- link link_5: geometry collision mesh filename=meshes/r1000ia80f/collision/link_5.stl; visual mesh filename=meshes/r1000ia80f/visual/link_5.stl
- link link_6: geometry collision mesh filename=meshes/r1000ia80f/collision/link_6.stl; visual mesh filename=meshes/r1000ia80f/visual/link_6.stl

File: rlbotics/envs/models/robots/universal_robots/ur10/ur10.urdf (robot description, URDF)
Before this commit: robot ur10, 11 links, 10 joints
Links:
- link base_link: geometry collision mesh filename=meshes/ur10/collision/base.stl; visual mesh filename=meshes/ur10/visual/base.dae
- link forearm_link: geometry collision mesh filename=meshes/ur10/collision/forearm.stl; visual mesh filename=meshes/ur10/visual/forearm.dae
- link shoulder_link: geometry collision mesh filename=meshes/ur10/collision/shoulder.stl; visual mesh filename=meshes/ur10/visual/shoulder.dae
- link upper_arm_link: geometry collision mesh filename=meshes/ur10/collision/upperarm.stl; visual mesh filename=meshes/ur10/visual/upperarm.dae
- link wrist_1_link: geometry collision mesh filename=meshes/ur10/collision/wrist1.stl; visual mesh filename=meshes/ur10/visual/wrist1.dae
- link wrist_2_link: geometry collision mesh filename=meshes/ur10/collision/wrist2.stl; visual mesh filename=meshes/ur10/visual/wrist2.dae
- link wrist_3_link: geometry collision mesh filename=meshes/ur10/collision/wrist3.stl; visual mesh filename=meshes/ur10/visual/wrist3.dae

File: rlbotics/envs/models/robots/universal_robots/ur3/ur3.urdf (robot description, URDF)
Before this commit: robot ur3, 11 links, 10 joints
Links:
- link base_link: geometry collision mesh filename=meshes/ur3/collision/base.stl; visual mesh filename=meshes/ur3/visual/base.dae
- link forearm_link: geometry collision mesh filename=meshes/ur3/collision/forearm.stl; visual mesh filename=meshes/ur3/visual/forearm.dae
- link shoulder_link: geometry collision mesh filename=meshes/ur3/collision/shoulder.stl; visual mesh filename=meshes/ur3/visual/shoulder.dae
- link upper_arm_link: geometry collision mesh filename=meshes/ur3/collision/upperarm.stl; visual mesh filename=meshes/ur3/visual/upperarm.dae
- link wrist_1_link: geometry collision mesh filename=meshes/ur3/collision/wrist1.stl; visual mesh filename=meshes/ur3/visual/wrist1.dae
- link wrist_2_link: geometry collision mesh filename=meshes/ur3/collision/wrist2.stl; visual mesh filename=meshes/ur3/visual/wrist2.dae
- link wrist_3_link: geometry collision mesh filename=meshes/ur3/collision/wrist3.stl; visual mesh filename=meshes/ur3/visual/wrist3.dae

File: rlbotics/envs/models/robots/universal_robots/ur5/ur5.urdf (robot description, URDF)
Before this commit: robot ur5, 11 links, 10 joints
Links:
- link base_link: geometry collision mesh filename=meshes/ur5/collision/base.stl; visual mesh filename=meshes/ur5/visual/base.dae
- link forearm_link: geometry collision mesh filename=meshes/ur5/collision/forearm.stl; visual mesh filename=meshes/ur5/visual/forearm.dae
- link shoulder_link: geometry collision mesh filename=meshes/ur5/collision/shoulder.stl; visual mesh filename=meshes/ur5/visual/shoulder.dae
- link upper_arm_link: geometry collision mesh filename=meshes/ur5/collision/upperarm.stl; visual mesh filename=meshes/ur5/visual/upperarm.dae
- link wrist_1_link: geometry collision mesh filename=meshes/ur5/collision/wrist1.stl; visual mesh filename=meshes/ur5/visual/wrist1.dae
- link wrist_2_link: geometry collision mesh filename=meshes/ur5/collision/wrist2.stl; visual mesh filename=meshes/ur5/visual/wrist2.dae
- link wrist_3_link: geometry collision mesh filename=meshes/ur5/collision/wrist3.stl; visual mesh filename=meshes/ur5/visual/wrist3.dae
