Commit message: mesh modification

File: rlbotics/envs/models/robots/kuka/kr210/kr210l150.urdf (robot description, URDF)
Before this commit: robot kuka_kr210, 9 links, 8 joints
Links:
- link base_link: geometry collision mesh filename=meshes/kr210l150/collision/base_link.stl; visual mesh filename=meshes/kr210l150/visual/base_link.stl
- link link_1: geometry collision mesh filename=meshes/kr210l150/collision/link_1.stl; visual mesh filename=meshes/kr210l150/visual/link_1.stl
- link link_2: geometry collision mesh filename=meshes/kr210l150/collision/link_2.stl; visual mesh filename=meshes/kr210l150/visual/link_2.stl
- link link_3: geometry collision mesh filename=meshes/kr210l150/collision/link_3.stl; visual mesh filename=meshes/kr210l150/visual/link_3.stl
- link link_4: geometry collision mesh filename=meshes/kr210l150/collision/link_4.stl; visual mesh filename=meshes/kr210l150/visual/link_4.stl
- link link_5: geometry collision mesh filename=meshes/kr210l150/collision/link_5.stl; visual mesh filename=meshes/kr210l150/visual/link_5.stl
- link link_6: geometry collision mesh filename=meshes/kr210l150/collision/link_6.stl; visual mesh filename=meshes/kr210l150/visual/link_6.stl
