Commit message: first welding torch and abb irb 5400 chaged mesh to stl

File: rlbotics/envs/models/robots/abb/irb5400/irb5400.urdf (robot description, URDF)
Before this commit: robot abb_irb5400, 10 links, 9 joints
Links:
- link base_link: geometry collision mesh filename=meshes/irb5400/collision/base_link.stl; visual mesh filename=meshes/irb5400/visual/base_link.stl
- link link_1: geometry collision mesh filename=meshes/irb5400/collision/link_1.stl; visual mesh filename=meshes/irb5400/visual/link_1.stl
- link link_2: geometry collision mesh filename=meshes/irb5400/collision/link_2.stl; visual mesh filename=meshes/irb5400/visual/link_2.stl
- link link_3: geometry collision mesh filename=meshes/irb5400/collision/link_3.stl; visual mesh filename=meshes/irb5400/visual/link_3.stl
- link link_4: geometry collision mesh filename=meshes/irb5400/collision/link_4.stl; visual mesh filename=meshes/irb5400/visual/link_4.stl
- link link_5: geometry collision mesh filename=meshes/irb5400/collision/link_5.stl; visual mesh filename=meshes/irb5400/visual/link_5.stl
- link link_5b: geometry collision mesh filename=meshes/irb5400/collision/link_5b.stl; visual mesh filename=meshes/irb5400/visual/link_5b.stl
- link link_6: geometry collision mesh filename=meshes/irb5400/collision/link_6.stl; visual mesh filename=meshes/irb5400/visual/link_6.stl
